File: test.sch (EAGLE design)
At the start: 2 parts, among them IC1 74ALS00D, IC2 MEGA16-A

Commit message: Verified ability of code in EagleFile can operate on schematic
git-svn-id: svn+ssh://bbfs-01.calit2.net/grw/Gordon/svn/trunk/Gadgets/Tools/EagleComposer@20771 2cf53259-273a-af40-bda6-69d31023b8ec
Other:
- note added: "print "Hello Eagle!" code_text_obj.text += "\n#Test!""
- note removed: "print "Hello Eagle!""
Changed lines of the file:
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@@
 <sheet>
 <plain>
-<text x="5.08" y="78.74" size="1.778" layer="213">print "Hello Eagle!"</text>
+<text x="5.08" y="78.74" size="1.778" layer="213">print "Hello Eagle!"
+code_text_obj.text += "\n#Test!"</text>
 </plain>
 <instances>
@@
 </schematic>
 </drawing>
+<compatibility>
+<note version="6.3" minversion="6.2.2" severity="warning">
+Since Version 6.2.2 text objects can contain more than one line,
+which will not be processed correctly with this version.
+</note>
+</compatibility>
 </eagle>
